File: kicad-stm32-cdaq.kicad_sch (KiCad schematic)
At the start: 0 parts

Commit message: Analog Inputs Sheet Completed
Changed lines of the file:
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@@
 	)
 	(sheet
-		(at 38.1 139.7)
+		(at 24.13 111.76)
 		(size 25.4 25.4)
 		(exclude_from_sim no)
@@
 		)
 		(property "Sheetname" "Power"
-			(at 38.1 138.9884 0)
+			(at 24.13 111.0484 0)
 			(effects
 				(font
@@
 		)
 		(property "Sheetfile" "power.kicad_sch"
-			(at 38.1 165.6846 0)
+			(at 24.13 137.7446 0)
 			(effects
 				(font
@@
 	(sheet
 		(at 25.4 25.4)
-		(size 19.05 25.4)
+		(size 25.4 25.4)
 		(exclude_from_sim no)
 		(in_bom yes)
@@
 		)
 		(pin "AIN0" output
-			(at 44.45 29.21 0)
+			(at 50.8 29.21 0)
 			(effects
 				(font
@@
 		)
 		(pin "AIN1" output
-			(at 44.45 31.75 0)
+			(at 50.8 31.75 0)
 			(effects
 				(font
@@
 		)
 		(pin "AIN2" output
-			(at 44.45 34.29 0)
+			(at 50.8 34.29 0)
 			(effects
 				(font
@@
 		)
 		(pin "AIN3" output
-			(at 44.45 36.83 0)
+			(at 50.8 36.83 0)
 			(effects
 				(font
@@
 		)
 		(pin "AIN4" output
-			(at 44.45 39.37 0)
+			(at 50.8 39.37 0)
 			(effects
 				(font
@@
 		)
 		(pin "AIN5" output
-			(at 44.45 41.91 0)
+			(at 50.8 41.91 0)
 			(effects
 				(font
@@
 		)
 		(pin "AIN6" output
-			(at 44.45 44.45 0)
+			(at 50.8 44.45 0)
 			(effects
 				(font
@@
 		)
 		(pin "AIN7" output
-			(at 44.45 46.99 0)
+			(at 50.8 46.99 0)
 			(effects
 				(font
