File: analog_inputs.kicad_sch (KiCad schematic)
At the start: 24 parts, among them J2 WJ500V-5.08-2P, J3 WJ500V-5.08-2P, J4 WJ500V-5.08-2P, J5 WJ500V-5.08-2P, J6 WJ500V-5.08-2P, J7 WJ500V-5.08-2P, J8 WJ500V-5.08-2P, J9 WJ500V-5.08-2P

Commit message: Analog Inputs Sheet Completed
Parts:
- removed R101, R102, R103, R104, R105, R106, R107: 100R, symbol Device:R
- added C201, C202, C203, C204, C205, C206, C207, C208: 10n, symbol Device:C
- added R202, R204, R206, R208, R213, R214, R215, R216: 6k8, symbol Device:R
- added R203, R205, R207, R209, R210, R211, R212: 150R, symbol Device:R
- R201: renamed from R100; value 100R -> 150R; LCSC Part # C122970 -> C870430; Mfr. Part # RT0603BRD07100RL -> RT1206BRD07150RL; Package 0603 -> 1206
Connections:
- net AIN0: now also C201.1, R202.2; no longer D200.1 (A1), J2.1 (Pin_1), R201.1
- net AIN1: now also C202.1, R204.2; no longer D201.1 (A1), J3.1 (Pin_1)
- net AIN2: now also C203.1, R206.2; no longer D202.1 (A1), J4.1 (Pin_1)
- net AIN3: now also C204.1, R208.2; no longer D203.1 (A1), J5.1 (Pin_1)
- net AIN4: now also C205.1, R213.2; no longer D204.1 (A1), J6.1 (Pin_1)
- net AIN5: now also C206.1, R214.2; no longer D205.1 (A1), J7.1 (Pin_1)
- net AIN6: now also C207.1, R215.2; no longer D206.1 (A1), J8.1 (Pin_1)
- net AIN7: now also C208.1, R216.2; no longer D207.1 (A1), J9.1 (Pin_1)
- net GND: now also C201.2, C202.2, C203.2, C204.2, C205.2, C206.2, C207.2, C208.2, R203.2, R205.2, R207.2, R209.2, R210.2, R211.2, R212.2
- new net: D207.1 (A1), J9.1 (Pin_1), R212.1, R216.1
- new net: D201.1 (A1), J3.1 (Pin_1), R203.1, R204.1
- new net: D200.1 (A1), J2.1 (Pin_1), R201.1, R202.1
- new net: D205.1 (A1), J7.1 (Pin_1), R210.1, R214.1
- new net: D202.1 (A1), J4.1 (Pin_1), R205.1, R206.1
- new net: D204.1 (A1), J6.1 (Pin_1), R209.1, R213.1
- new net: D206.1 (A1), J8.1 (Pin_1), R211.1, R215.1
- new net: D203.1 (A1), J5.1 (Pin_1), R207.1, R208.1
Other:
- note added: "0.1% 25ppm/ºC 1206"
- note added: "0.1% 25ppm/ºC 1206 POT = 22mA * 22mA * 150R * 2 = 145.2mW"
- note added: "AN2834"
- note added: "Connectors + TVS + Current to Voltage Converter"
- note added: "FAIN <= 1470Hz (>500Hz)"
- note added: "FC @ -3db = 2400Hz"
- note added: "VMAX = 150R . 22mA = 3.3V VRWM = 3.3V IR = 200nA (<< 3.6mA) 4V < VBR @ 1mA < 6V VCLAMP = 12V (Smallest)"
- note removed: "0.1% 25ppm/ºC"
- note removed: "Connectors + TVS + I->V"
- note removed: "VMAX = 100R . 21mA = 2.1V VMIN = 100R . 3.6mA = 0.36V VRWM = 3.3V (> 2.1V) IR = 200nA (<< 3.6mA) 4V < VBR @ 1mA < 6V VCLAMP = 12V (Smallest)"

Commit message: Extra comments
Other:
- note added: "Connectors + TVS + Current to Voltage Converter + LPF"
- note added: "STM32F407xx RAINMAX = 50k R = 6k8 (< 50K)"
- note removed: "Connectors + TVS + Current to Voltage Converter"
Changed lines of the file:
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@@
 	(text "FAIN <= 1470Hz (>500Hz)"
 		(exclude_from_sim no)
-		(at 241.3 144.78 0)
+		(at 241.3 158.75 0)
+		(effects
+			(font
+				(size 1.27 1.27)
+			)
+			(justify left top)
+		)
+	)
+	(text "STM32F407xx\n\nRAINMAX = 50k\n\nR = 6k8 (< 50K)"
+		(exclude_from_sim no)
+		(at 246.38 134.62 0)
 		(effects
 			(font
@@
 		)
 	)
-	(text "Connectors + TVS + Current to Voltage Converter"
+	(text "Connectors + TVS + Current to Voltage Converter + LPF"
 		(exclude_from_sim no)
 		(at 13.97 26.67 0)
@@
 	(text "AN2834"
 		(exclude_from_sim no)
-		(at 250.19 134.62 0)
+		(at 250.19 148.59 0)
 		(effects
 			(font
@@
 	)
 	(image
-		(at 255.27 139.7)
+		(at 255.27 153.67)
 		(scale 0.360553)
 		(data "iVBORw0KGgoAAAANSUhEUgAAATgAAAA5CAIAAAAtNqAsAAAAA3NCSVQICAjb4U/gAAAACXBIWXMA"
